File: M.2_Slot_Oculink/M.2_Slot_Oculink.kicad_sch (KiCad schematic)
At the start: 0 parts

Commit message: Update
Parts:
- added J1: Bus_M.2_Socket_M, symbol Connector:Bus_M.2_Socket_M
- added J2: Oculink, 1719820142:1719820142, symbol 1719820142:1719820142
Connections:
- new net +3V3: J1.12 (3.3V), J1.14 (3.3V), J1.16 (3.3V), J1.18 (3.3V), J1.2 (3.3V), J1.4 (3.3V), J1.70 (3.3V), J1.72 (3.3V), J1.74 (3.3V)
- new net CLCK+: J1.55 (REFCLKp), J2.B12
- new net CLCK-: J1.53 (REFCLKn), J2.B13
- new net GND: J1.1 (GND), J1.15 (GND), J1.21 (GND), J1.27 (GND), J1.3 (GND), J1.33 (GND), J1.39 (GND), J1.45 (GND), J1.51 (GND), J1.57 (GND), J1.71 (GND), J1.73 (GND), J1.75 (GND), J1.9 (GND)
- new net RX+0: J1.43 (PERp0/SATA-B-), J2.B3
- new net RX+1: J1.31 (PERp1), J2.B6
- new net RX+2: J1.19 (PERp2), J2.B15
- new net RX+3: J1.7 (PERp3), J2.B18
- new net RX-0: J1.41 (PERn0/SATA-B+), J2.B4
- new net RX-1: J1.29 (PERn1), J2.B7
- new net RX-2: J1.17 (PERn2), J2.B16
- new net RX-3: J1.5 (PERn3), J2.B19
- new net TX+0: J1.49 (PETp0/SATA-A+), J2.A3
- new net TX+1: J1.37 (PETp1), J2.A6
- new net TX+2: J1.25 (PETp2), J2.A15
- new net TX+3: J1.13 (PETp3), J2.A18
- new net TX-0: J1.47 (PETn0/SATA-A-), J2.A4
- new net TX-1: J1.35 (PETn1), J2.A7
- new net TX-2: J1.23 (PETn2), J2.A16
- new net TX-3: J1.11 (PETn3), J2.A19
