File: Oculink_Dock/Oculink_Dock.kicad_sch (KiCad schematic)
At the start: 8 parts, among them J1 Bus_M.2_Socket_M, J2 Oculink

Commit message: Update
Parts:
- removed C1, C2, C3, C4: 100nF, Capacitor_SMD:C_0603_1608Metric, symbol Device:C
- removed D1: G, LED_SMD:LED_0603_1608Metric, symbol Device:LED
- removed J1: Bus_M.2_Socket_M, symbol Connector:Bus_M.2_Socket_M
- removed J2: Oculink, 1719820142:1719820142, symbol 1719820142:1719820142
- removed R1: 100, Resistor_SMD:R_0603_1608Metric, symbol Device:R
- added J1: 1719820142, 1719820142:1719820142, symbol 1719820142:1719820142
- added J3: ERF8-025-XX-X-D-RA-L-XX, ERF8-025-XX-X-D-RA-L-XX:SAMTEC_ERF8-025-XX-X-D-RA-L-XX, symbol ERF8-025-XX-X-D-RA-L-XX:ERF8-025-XX-X-D-RA-L-XX
- added J4: DIN-4, Package_SO:TSSOP-20_4.4x6.5mm_P0.65mm, symbol Connector:DIN-4
Connections:
- net +3V3: now also J1.A1, J1.B21
- net GND: now also J1.A11, J1.A14, J1.A17, J1.A2, J1.A20, J1.A5, J1.A8, J1.B11, J1.B14, J1.B17, J1.B2, J1.B20, J1.B5, J1.B8, J1.MP1, J1.MP2, J1.MP3, J1.MP4, J4.2, J4.3
- net PERST: now also J1.A12
- new net +12V: J4.1, J4.4
- new net +5V: J1.A21, J1.B1
- new net BP_TYPE: J1.B9
- new net CLK: J1.A9
- new net CPRSNT: J1.A13
- new net CWAKE: J1.B10
- new net DATA: J1.A10
- new net REFCLK+: J1.B12
- new net REFCLK-: J1.B13
- new net RX0+: J1.A3
- new net RX0-: J1.A4
- new net RX1+: J1.A6
- new net RX1-: J1.A7
- new net RX2+: J1.A15
- new net RX2-: J1.A16
- new net RX3+: J1.A18
- new net RX3-: J1.A19
- new net TX0+: J1.B3
- new net TX0-: J1.B4
- new net TX1+: J1.B6
- new net TX1-: J1.B7
- new net TX2+: J1.B15
- new net TX2-: J1.B16
- new net TX3+: J1.B18
- new net TX3-: J1.B19
- no-connect marks 1 -> 0

Commit message: Update
Parts:
- added Presence: Conn_01x01_Pin, symbol Connector:Conn_01x01_Pin
- added SW2: Eject, Button_Switch_SMD:Nidec_Copal_CAS-120A, symbol Switch:SW_Push
- added SW3: Rescan, Button_Switch_SMD:Nidec_Copal_CAS-120A, symbol Switch:SW_Push
Connections:
- net +3V3: now also J3.01, J3.38
- net +5V: now also J3.41, J3.43
- net BP_TYPE: now also J3.14
- net CLK: now also J3.17
- net CPRSNT: now also J3.25
- net CWAKE: now also J3.16
- net DATA: now also J3.19
- net GND: now also J3.03, J3.06, J3.09, J3.12, J3.15, J3.18, J3.21, J3.24, J3.27, J3.30, J3.33, J3.36, J3.39, J3.40, J3.42, J3.44, J3.45, J3.46
- net PERST: now also J3.23
- net REFCLK+: now also J3.20
- net REFCLK-: now also J3.22
- net RX0+: now also J3.05
- net RX0-: now also J3.07
- net RX1+: now also J3.11
- net RX1-: now also J3.13
- net RX2+: now also J3.29
- net RX2-: now also J3.31
- net RX3+: now also J3.35
- net RX3-: now also J3.37
- net TX0+: now also J3.02
- net TX0-: now also J3.04
- net TX1+: now also J3.08
- net TX1-: now also J3.10
- net TX2+: now also J3.26
- net TX2-: now also J3.28
- net TX3+: now also J3.32
- net TX3-: now also J3.34
- new net PRSNC: Presence.1 (Pin_1)
Other:
- added sheet DevBoard (devboard.kicad_sch)

Commit message: Update
Parts:
- added C18, C19: 10uF, symbol Device:C
- added C20, C22: 100nF, symbol Device:C
- added C21: 22nF, symbol Device:C
- added C23, C24: 15uF, symbol Device:C
- added C25: 150pF, symbol Device:C
- added L1: 2.2uH, symbol Device:L
- added R10: 45.3k, symbol Device:R
- added R11: 10k, symbol Device:R
- added R8: 52.3k, symbol Device:R
- added R9: 100k, symbol Device:R
- added U4: TPS259470ARPWR, RPW0010A-MFG, symbol TPS259470ARPWR:TPS259470ARPWR
- added U5: TPS56A37RPAR, RPA0010A-MFG, symbol TPS56A37RPAR:TPS56A37RPAR
Connections:
- net GND is gone; now on net +12V: J1.A11, J1.A14, J1.A17, J1.A2, J1.A20, J1.A5, J1.A8, J1.B11, J1.B14, J1.B17, J1.B2, J1.B20, J1.B5, J1.B8, J1.MP1, J1.MP2, J1.MP3, J1.MP4, J3.03, J3.06, J3.09, J3.12, J3.15, J3.18, J3.21, J3.24, J3.27, J3.30, J3.33, J3.36, J3.39, J3.40, J3.42, J3.44, J3.45, J3.46, J4.2, J4.3
- net +12V: now also J3.01, J3.38, C18.1, C19.2, C20.1, C20.2, C21.2, C23.1, C24.2, C25.1, L1.2, R10.2, R11.1, R8.2, U4.5 (IN), U5.3 (AGND), U5.8 (VIN), U5.9 (PGND)
- net +5V: no longer J1.A21, J1.B1
- net +3V3 renamed O_3v3
- net O_3v3: no longer J3.01, J3.38
- new net: R8.1, U5.10 (MODE)
- new net: C25.2, R10.1, R11.2, U5.2 (FB)
- new net: R9.1, U5.4 (PG)
- new net: C21.1, U5.5 (SS)
- new net: C22.2, L1.1, U5.6 (SW)
- new net: C22.1, U5.7 (BOOT)
- new net: C23.2, C24.1
- new net: C18.2, C19.1
- new net 3.3v: R9.2
- new net O_5v: J1.A21, J1.B1
- new net PCIe_PWR: U4.6 (OUT)
- no-connect marks 0 -> 1
Other:
- moved on the sheet: SW2, SW3

Commit message: Update
Parts:
- added C13: 1uF, symbol Device:C
- added C14: 2.2nF, symbol Device:C
- added C26: 3300pF, symbol Device:C
- added C27: 470uF, symbol Device:C
- added D1: D_Zener, Package_CSP:OnSemi_ODCSP8_BGA-8_3.16x3.16mm_Layout3x3_P1.26mm, symbol Device:D_Zener
- added D2: D_Schottky, symbol Device:D_Schottky
- added R1: 470k, symbol Device:R
- added R12, R14: 47k, symbol Device:R
- added R13: 549, symbol Device:R
- added R15: 5.6k, symbol Device:R
- added R16: 390k, symbol Device:R
- added R17: 100k, symbol Device:R
- added U2: INA219BxDCN, Package_TO_SOT_SMD:SOT-23-8, symbol Sensor_Energy:INA219BxDCN
Connections:
- net +5V is gone; now on net PCIe_PWR: J3.41, J3.43
- net 3.3v is gone; now on net +12V: R9.2
- net +12V: now also SW2.1, SW3.1, U4.8 (GND), C13.1, C13.2, C14.2, C26.2, C27.2, D1.1 (K), D1.2 (A), D2.2 (A), R1.1, R12.1, R13.2, R15.2, R16.1, R17.2; no longer J3.42, J3.44, J3.45, J3.46
- net PCIe_PWR: now also J3.42, J3.44, J3.45, J3.46, J3.47, J3.48, C27.1, D2.1 (K), R14.1
- net at U4.1 (EN_UVLO): now also R1.2, R12.2
- net at U4.10 (ITIMER): now also C14.1
- net at U4.2 (OVCSEL): now also R16.2
- net at U4.3 (PG): now also R17.1
- net at U4.4 (PGTH): now also R14.2, R15.1
- net at U4.7 (dVdt): now also C26.1
- net at U4.9 (ILM): now also R13.1
- net G3: now reaches SW2.2
- net G2: now reaches SW3.2
Other:
- moved on the sheet: J1, SW2, U4

Commit message: Update
Parts:
- added J2: Screen, Display:NHD-C0220BiZ-FSRGB, symbol Connector_Generic:Conn_01x08
- added R18, R2: 0.03, symbol Device:R
- added SW4: RotaryEncoder_Switch, symbol Device:RotaryEncoder_Switch
- added U6: INA219BxDCN, Package_TO_SOT_SMD:SOT-23-8, symbol Sensor_Energy:INA219BxDCN
Connections:
- net +12V: now also U2.2 (IN-), U2.3 (GND), U2.7 (A0), U2.8 (A1), J2.2 (Pin_2), R2.1, SW4.C, SW4.S2, U6.3 (GND), U6.7 (A0); no longer J3.01, J3.38, R17.2, R9.2
- net PCIe_PWR: now also R18.1, U6.1 (IN+); no longer C27.1, D2.1 (K), R14.1, U4.6 (OUT)
- net +3V3: now reaches U2.1 (IN+)
- net +3V3: now also J3.01, J3.38, R17.2, R9.2, U2.4 (VS), J2.1 (Pin_1), R2.2, U6.4 (VS), U6.8 (A1)
- net G5: now reaches U2.5 (SCL)
- net G5: now also U6.5 (SCL)
- net G4: now reaches U2.6 (SDA)
- net G4: now also U6.6 (SDA)
- net PRSNC renamed G6
- new net: C27.1, D2.1 (K), R14.1, R18.2, U4.6 (OUT), U6.2 (IN-)
- new net G10: J2.3 (Pin_3)
- new net G11: J2.4 (Pin_4)
- new net G12: J2.6 (Pin_6)
- new net G13: J2.7 (Pin_7)
- new net G14: J2.8 (Pin_8)
- new net G15: SW4.A
- new net G16: SW4.B
- new net G17: SW4.S1
- new net G9: J2.5 (Pin_5)
Other:
- moved on the sheet: U2

Commit message: Update
Parts:
- J1: renamed from Presence; value Conn_01x01_Pin -> Prsnc
- renumbered C18 to C1, C23 to C10, C24 to C11, C27 to C12, C19 to C2, C20 to C3, C21 to C4, C13 to C5, C14 to C6, C26 to C7, C22 to C8, C25 to C9, J1 to J5, R12 to R1, R14 to R10, R15 to R11, R2 to R12, R18 to R13, R16 to R2, R8 to R3, R1 to R4, R9 to R5, R17 to R6, R10 to R7, R11 to R8, R13 to R9, SW4 to SW1, U5 to U1, U4 to U2, U2 to U3, U6 to U4
Connections:
- net +12V: now also J3.45, J3.46
- net PCIe_PWR: now also J3.49, J3.50; no longer J3.45, J3.46
- net G0: now reaches R5.1, U1.4 (PG)
- net G1: now reaches R6.1, U2.3 (PG)

Commit message: Update
Parts:
- added D3, D4: LED, LED_SMD:LED_Cree-XHP50_3V_HighDensity, symbol Device:LED
- added R21, R23: 2.2k, symbol Device:R
Connections:
- net +12V: no longer C10.1, C11.2, C12.2, C2.2, C3.2, C4.2, C5.2, C6.2, C7.2, C9.1, D1.2 (A), D2.2 (A), J2.2 (Pin_2), J3.03, J3.06, J3.09, J3.12, J3.15, J3.18, J3.21, J3.24, J3.27, J3.30, J3.33, J3.36, J3.39, J3.40, J3.45, J3.46, J4.2, J4.3, J5.A11, J5.A14, J5.A17, J5.A2, J5.A20, J5.A5, J5.A8, J5.B11, J5.B14, J5.B17, J5.B2, J5.B20, J5.B5, J5.B8, J5.MP1, J5.MP2, J5.MP3, J5.MP4, L1.2, R1.1, R11.2, R12.1, R2.1, R3.2, R7.2, R8.1, R9.2, SW1.C, SW1.S2, SW2.1, SW3.1, U1.3 (AGND), U1.9 (PGND), U2.8 (GND), U3.2 (IN-), U3.3 (GND), U3.7 (A0), U3.8 (A1), U4.3 (GND), U4.7 (A0)
- net +3V3: now also R23.1
- new net: D4.1 (K), R23.2
- new net: D3.1 (K), R21.2
- new net GND: C10.1, C11.2, C12.2, C2.2, C3.2, C4.2, C5.2, C6.2, C7.2, C9.1, D1.2 (A), D2.2 (A), D3.2 (A), D4.2 (A), J2.2 (Pin_2), J3.03, J3.06, J3.09, J3.12, J3.15, J3.18, J3.21, J3.24, J3.27, J3.30, J3.33, J3.36, J3.39, J3.40, J3.45, J3.46, J4.2, J4.3, J5.A11, J5.A14, J5.A17, J5.A2, J5.A20, J5.A5, J5.A8, J5.B11, J5.B14, J5.B17, J5.B2, J5.B20, J5.B5, J5.B8, J5.MP1, J5.MP2, J5.MP3, J5.MP4, L1.2, R1.1, R11.2, R12.1, R2.1, R3.2, R7.2, R8.1, R9.2, SW1.C, SW1.S2, SW2.1, SW3.1, U1.3 (AGND), U1.9 (PGND), U2.8 (GND), U3.2 (IN-), U3.3 (GND), U3.7 (A0), U3.8 (A1), U4.3 (GND), U4.7 (A0)
- new net USB_VBUS: R21.1

Commit message: Update
Parts:
- added R24, R25, R26, R27: 2.2k, Resistor_SMD:R_0805_2012Metric, symbol Device:R
- C1, C10, C11, C2, C3, C4, C5, C6, C7, C8, C9: footprint (none) -> Capacitor_SMD:C_0805_2012Metric
- C12: footprint (none) -> Capacitor_SMD:CP_Elec_8x10
- D2: footprint (none) -> Diode_SMD:D_SMB
- J1: footprint (none) -> Connector_PinHeader_2.54mm:PinHeader_1x01_P2.54mm_Horizontal
- J3: footprint ERF8-025-XX-X-D-RA-L-XX:SAMTEC_ERF8-025-XX-X-D-RA-L-XX -> Connector_Samtec_EdgeRate:Samtec_ERF8-025-XX.X-DV-L_2x25_P0.8mm_Socket_Latch
- L1: footprint (none) -> Inductor_SMD:L_10.4x10.4_H4.8
- R1: value 47k -> 59k; footprint (none) -> Resistor_SMD:R_0805_2012Metric
- R10, R11, R2, R21, R23, R3, R4, R5, R6, R7, R8, R9: footprint (none) -> Resistor_SMD:R_0805_2012Metric
- R12, R13: footprint (none) -> Resistor_SMD:R_1206_3216Metric
- SW1: footprint (none) -> Rotary_Encoder:RotaryEncoder_Alps_EC12E-Switch_Vertical_H20mm
- U1: footprint RPA0010A-MFG -> TPS56A37RPAR:RPA0010A-MFG
- U2: footprint RPW0010A-MFG -> TPS259470ARPWR:RPW0010A-MFG
Connections:
- net +12V: now also C2.1
- net +3V3: now also R24.1, R25.1, R26.1, R27.1
- net G4: now also R24.2, R27.2
- net G5: now also R25.2, R26.2
- net GND: now also C1.2, C10.2, C11.1, D3.1 (K), D4.1 (K); no longer D3.2 (A), D4.2 (A)
- net at R23.2: now also D4.2 (A); no longer D4.1 (K)
- net at R21.2: now also D3.2 (A); no longer D3.1 (K)
Other:
- moved on the sheet: C11, C2, D3, D4
