File: Oculink_Dock/devboard.kicad_sch (KiCad schematic)
At the start: 34 parts, among them J2 USB_C_Receptacle_USB2.0_14P, J5 Conn_01x10, J6 Conn_01x10, J7 Conn_01x10, J8 Conn_01x03, SW1 SW_Push, U1 RP2040, U2 NCP1117-3.3_SOT223, U3 W25Q128JVS, Y1 12 MHz

Commit message: Update
Parts:
- removed C13, C14: 10uF, symbol Device:C
- removed J2: USB_C_Receptacle_USB2.0_14P, Package_DFN_QFN:QFN-56-1EP_7x7mm_P0.4mm_EP3.2x3.2mm, symbol Connector:USB_C_Receptacle_USB2.0_14P
- removed R1, R2: 5.1k, symbol Device:R
- removed U2: NCP1117-3.3_SOT223, Package_TO_SOT_SMD:SOT-223-3_TabPin2, symbol Regulator_Linear:NCP1117-3.3_SOT223

Commit message: Update
Parts:
- removed J5: Conn_01x10, symbol Connector_Generic:Conn_01x10
- renumbered C17 to C13, C1 to C14, C2 to C17, C3 to C18, C4 to C19, C5 to C20, C6 to C21, C7 to C22, C8 to C23, C9 to C24, C10 to C25, C11 to C26, C12 to C27, J8 to J6, J6 to J7, J7 to J8, R7 to R14, R3 to R15, R4 to R16, R6 to R17, R5 to R18, SW1 to SW4, U3 to U5, U1 to U6
Connections:
- net G10: no longer J7.1 (Pin_1)
- net G11: no longer J7.2 (Pin_2)
- net G12: no longer J7.3 (Pin_3)
- net G13: no longer J7.4 (Pin_4)
- net G14: no longer J7.5 (Pin_5)
- net G15: no longer J7.6 (Pin_6)
- net G16: no longer J7.7 (Pin_7)
- net G17: no longer J7.8 (Pin_8)
- net G7: now also J7.7 (Pin_7)
- net G8: now also J7.8 (Pin_8)
- no-connect marks 0 -> 6

Commit message: Update
Parts:
- added J9: USB_C_Receptacle_USB2.0_14P, Package_DFN_QFN:WDFN-10-1EP_3x3mm_P0.5mm_EP1.8x2.5mm, symbol Connector:USB_C_Receptacle_USB2.0_14P
- added R19, R20: 5.1k, symbol Device:R
Connections:
- net D+: now also J9.A6 (D+), J9.B6 (D+)
- net D-: now also J9.A7 (D-), J9.B7 (D-)
- net GND: now also R19.2, R20.2
- new net: J9.A5 (CC1), R19.1
- new net: J9.B5 (CC2), R20.1
- new net: J9.A1 (GND), J9.A12 (GND), J9.B1 (GND), J9.B12 (GND)
- new net: J9.A4 (VBUS), J9.A9 (VBUS), J9.B4 (VBUS), J9.B9 (VBUS)

Commit message: Update
Parts:
- added C28: 100nF, symbol Device:C
- added R22: 10k, symbol Device:R
- added SW5: SW_Push, PCM_marbastlib-he:SW_MX_HE_0deg_1u, symbol Switch:SW_Push
Connections:
- net +3V3: now also R22.1
- net GND: now also J9.A1 (GND), J9.A12 (GND), J9.B1 (GND), J9.B12 (GND), J9.SH (SHIELD), C28.1, SW5.1
- net USB_VBUS: now reaches J9.A4 (VBUS), J9.A9 (VBUS), J9.B4 (VBUS), J9.B9 (VBUS)
- net RUN: no longer names the net of U6.26 (RUN)
- net RUN: now also R22.2, SW5.2
- net TESTEN: no longer names the net of U6.19 (TESTEN)
- net TESTEN: now also C28.2

Commit message: Update
Parts:
- removed C28: 100nF, symbol Device:C
- removed J7: Conn_01x10, symbol Connector_Generic:Conn_01x10
- added J10: Conn_01x04, Connector_PinHeader_2.54mm:PinHeader_1x04_P2.54mm_Vertical, symbol Connector_Generic:Conn_01x04
- C13, C14, C15, C16, C17, C18, C19, C20, C21, C22, C23, C24, C25, C26, C27: footprint (none) -> Capacitor_SMD:C_0805_2012Metric
- J6: footprint Oscillator:Oscillator_DIP-14 -> Connector_PinHeader_2.54mm:PinHeader_1x03_P2.54mm_Vertical
- J8: footprint (none) -> Connector_PinHeader_2.54mm:PinHeader_1x10_P2.54mm_Vertical
- R14, R17: footprint Package_SO:SOIC-8_5.3x5.3mm_P1.27mm -> Resistor_SMD:R_0805_2012Metric
- R15, R16, R18, R19, R20, R22: footprint (none) -> Resistor_SMD:R_0805_2012Metric
Connections:
- net G18: now also J10.3 (Pin_3)
- net G19: now also J10.4 (Pin_4)
- net G7: now also J10.1 (Pin_1)
- net G8: now also J10.2 (Pin_2)
- net GND: now also U6.19 (TESTEN)
- no-connect marks 6 -> 0
